Commit message: Updated arm base link mass for stability in gazebo

File: kinova_arm_description/description/kinova_arm.urdf.xacro (robot description, xacro)
@@ -16,7 +16,7 @@
     <link name="arm_base_link">
         <inertial>
-            <mass value="10.0"/>
+            <mass value="50.0"/>
             <origin xyz="0 0 0" rpy="0 0 0"/>
-            <inertia ixx="1.0" ixy="0" ixz="0" iyy="1.0" iyz="0" izz="1.0"/>
+            <inertia ixx="5.0" ixy="0" ixz="0" iyy="5.0" iyz="0" izz="5.0"/>
         </inertial>
     </link>
